File: Motor_Shield/Motor_Shield.kicad_pcb (KiCad board)
At the start: 2 copper layers, 50 parts, among them J1 Conn_01x08_Female, J2 Conn_01x06_Female, J3 Conn_01x08_Female, J4 Conn_01x10_Female, J5 Conn_01x02_Female, J6 Screw_Terminal_01x06, U1 L6474PD

Commit message: Pcb fertig aber noch nicht optimal
Parts:
- removed R17: NP, Resistor_SMD:R_1206_3216Metric_Pad1.42x1.75mm_HandSolder
- C1, C10, C2, C4, C5, C7, C8, C9, D1, D2, D3, D4, D5, D6, D7, R1, R10, R11, R12, R13, R14, R15, R16, R18, R19, R2, R20, R21, R22, R23, R24, R25, R3, R4, R5, R6, R7, R8, R9, U1: moved to B.Cu
- C3, C6: footprint Capacitor_Tantalum_SMD:CP_EIA-7260-38_AVX-R_Pad2.68x6.30mm_HandSolder -> Capacitor_Tantalum_SMD:CP_EIA-3528-12_Kemet-T_Pad1.50x2.35mm_HandSolder; moved to B.Cu
- moved J1 67.2 mm to (175.3, 91.9)
- moved J2 67.2 mm to (175.3, 74.2)
- moved J3 67.2 mm to (126.7, 74.2)
- moved J4 67.2 mm to (126.7, 96.0)
- moved R2 49.8 mm to (122.1, 79.2), turned to 180 degrees
- moved R7 49.8 mm to (130.0, 99.6), turned to 90 degrees
- moved R10 49.4 mm to (121.9, 89.4), turned to 180 degrees
- moved J5 48.2 mm to (134.1, 103.1)
- moved R13 45.0 mm to (138.7, 108.2)
- moved C11 43.9 mm to (138.7, 97.5), turned to 90 degrees
- moved R12 43.6 mm to (130.3, 111.5), turned to 270 degrees
- moved R9 38.5 mm to (121.9, 86.9), turned to 180 degrees
- moved R1 37.3 mm to (130.6, 74.0), turned to 90 degrees
- moved C1 37.1 mm to (170.5, 85.2)
- moved R4 36.4 mm to (133.1, 86.4)
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Routing:
- net GND: track 0.00 -> 326.7 mm
- net VDD: track 0.00 -> 188.6 mm, vias 0 -> 2
- net Net-(R6-Pad1): track 0.00 -> 142.3 mm, vias 0 -> 6
- net Net-(R11-Pad2): track 0.00 -> 116.1 mm, vias 0 -> 8
- net VS: track 0.00 -> 115.7 mm, vias 0 -> 8
- net Net-(D6-Pad2): track 0.00 -> 105.2 mm
- net Net-(R13-Pad2): track 0.00 -> 84.4 mm, vias 0 -> 8
- net Net-(R19-Pad2): track 0.00 -> 71.1 mm, vias 0 -> 4
- net Net-(D4-Pad2): track 0.00 -> 68.1 mm, vias 0 -> 2
- net Net-(D7-Pad2): track 0.00 -> 65.2 mm, vias 0 -> 2
- net Net-(R10-Pad2): track 0.00 -> 58.9 mm, vias 0 -> 2
- net Net-(C2-Pad1): track 0.00 -> 46.6 mm, vias 0 -> 2
- net Net-(D5-Pad2): track 0.00 -> 40.3 mm
- net Net-(D1-Pad1): track 0.00 -> 37.9 mm, vias 0 -> 2
- net Net-(R14-Pad1): track 0.00 -> 34.6 mm, vias 0 -> 2
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- added copper zone on B.Cu, net GND
Other:
- board outline added: 65.4 x 65.4 mm
