File: Motor_Shield/Motor_Shield.sch (KiCad schematic (older format))
At the start: 50 parts, among them J1 Conn_01x08_Female, J2 Conn_01x06_Female, J3 Conn_01x08_Female, J4 Conn_01x10_Female, J5 Conn_01x02_Female, J6 Screw_Terminal_01x06, U1 L6474PD

Commit message: Pcb fertig aber noch nicht optimal
Parts:
- removed R17: NP, Resistor_SMD:R_1206_3216Metric_Pad1.42x1.75mm_HandSolder, symbol Device:R
- C3, C6: footprint Capacitor_Tantalum_SMD:CP_EIA-7260-38_AVX-R_Pad2.68x6.30mm_HandSolder -> Capacitor_Tantalum_SMD:CP_EIA-3528-12_Kemet-T_Pad1.50x2.35mm_HandSolder
Connections:
- no-connect marks 0 -> 2
Other:
- moved on the sheet: C3, C5, D2, R18
Changed lines of the file:
@@
 L Device:C C5
 U 1 1 5E578ABE
-P 4800 1400
-F 0 "C5" H 4915 1446 50  0000 L CNN
-F 1 "100nF" H 4915 1355 50  0000 L CNN
-F 2 "Capacitor_SMD:C_1206_3216Metric_Pad1.42x1.75mm_HandSolder" H 4838 1250 50  0001 C CNN
-F 3 "~" H 4800 1400 50  0001 C CNN
-	1    4800 1400
+P 4100 1400
+F 0 "C5" H 4215 1446 50  0000 L CNN
+F 1 "100nF" H 4215 1355 50  0000 L CNN
+F 2 "Capacitor_SMD:C_1206_3216Metric_Pad1.42x1.75mm_HandSolder" H 4138 1250 50  0001 C CNN
+F 3 "~" H 4100 1400 50  0001 C CNN
+	1    4100 1400
 	1    0    0    -1
 $EndComp
@@
 L Device:CP C3
 U 1 1 5E579F35
-P 4350 1400
-F 0 "C3" H 4468 1446 50  0000 L CNN
-F 1 "47uF" H 4468 1355 50  0000 L CNN
-F 2 "Capacitor_Tantalum_SMD:CP_EIA-7260-38_AVX-R_Pad2.68x6.30mm_HandSolder" H 4388 1250 50  0001 C CNN
-F 3 "~" H 4350 1400 50  0001 C CNN
-	1    4350 1400
+P 3650 1400
+F 0 "C3" H 3768 1446 50  0000 L CNN
+F 1 "47uF" H 3768 1355 50  0000 L CNN
+F 2 "Capacitor_Tantalum_SMD:CP_EIA-3528-12_Kemet-T_Pad1.50x2.35mm_HandSolder" H 3688 1250 50  0001 C CNN
+F 3 "~" H 3650 1400 50  0001 C CNN
+	1    3650 1400
 	1    0    0    -1
 $EndComp
@@
 L Device:LED D2
 U 1 1 5E57AFA2
-P 3800 1400
-F 0 "D2" V 3839 1283 50  0000 R CNN
-F 1 "LED" V 3748 1283 50  0000 R CNN
-F 2 "Diode_SMD:D_1206_3216Metric_Pad1.42x1.75mm_HandSolder" H 3800 1400 50  0001 C CNN
-F 3 "~" H 3800 1400 50  0001 C CNN
-	1    3800 1400
+P 3100 1400
+F 0 "D2" V 3139 1283 50  0000 R CNN
+F 1 "LED" V 3048 1283 50  0000 R CNN
+F 2 "Diode_SMD:D_1206_3216Metric_Pad1.42x1.75mm_HandSolder" H 3100 1400 50  0001 C CNN
+F 3 "~" H 3100 1400 50  0001 C CNN
+	1    3100 1400
 	0    -1   -1   0
 $EndComp
@@
 L Device:R R18
 U 1 1 5E57C0FF
-P 4650 1050
-F 0 "R18" V 4443 1050 50  0000 C CNN
-F 1 "330" V 4534 1050 50  0000 C CNN
-F 2 "Resistor_SMD:R_1206_3216Metric_Pad1.42x1.75mm_HandSolder" V 4580 1050 50  0001 C CNN
-F 3 "~" H 4650 1050 50  0001 C CNN
-	1    4650 1050
+P 3950 1050
+F 0 "R18" V 3743 1050 50  0000 C CNN
+F 1 "330" V 3834 1050 50  0000 C CNN
+F 2 "Resistor_SMD:R_1206_3216Metric_Pad1.42x1.75mm_HandSolder" V 3880 1050 50  0001 C CNN
+F 3 "~" H 3950 1050 50  0001 C CNN
+	1    3950 1050
 	0    1    1    0
 $EndComp
 Wire Wire Line
-	3800 1250 3800 1050
-Wire Wire Line
-	5300 1050 5300 1250
-Wire Wire Line
-	5300 1700 5450 1700
+	3100 1250 3100 1050
+Wire Wire Line
+	4600 1050 4600 1250
 Wire Wire Line
 	5450 1700 5450 2400
 Wire Wire Line
-	4800 1050 5300 1050
-Connection ~ 5300 1250
-Wire Wire Line
-	5300 1250 5300 1700
-Wire Wire Line
-	4800 1250 5300 1250
+	4100 1050 4600 1050
+Connection ~ 4600 1250
+Wire Wire Line
+	4600 1250 4600 1700
+Wire Wire Line
+	4100 1250 4600 1250
 $Comp
 L power:GND #PWR08
 U 1 1 5E57F0F0
-P 3800 1650
-F 0 "#PWR08" H 3800 1400 50  0001 C CNN
-F 1 "GND" H 3805 1477 50  0000 C CNN
-F 2 "" H 3800 1650 50  0001 C CNN
-F 3 "" H 3800 1650 50  0001 C CNN
-	1    3800 1650
+P 3100 1650
+F 0 "#PWR08" H 3100 1400 50  0001 C CNN
+F 1 "GND" H 3105 1477 50  0000 C CNN
+F 2 "" H 3100 1650 50  0001 C CNN
+F 3 "" H 3100 1650 50  0001 C CNN
+	1    3100 1650
 	1    0    0    -1
 $EndComp
@@
 L power:GND #PWR010
 U 1 1 5E57FA7B
-P 4350 1650
-F 0 "#PWR010" H 4350 1400 50  0001 C CNN
-F 1 "GND" H 4355 1477 50  0000 C CNN
-F 2 "" H 4350 1650 50  0001 C CNN
-F 3 "" H 4350 1650 50  0001 C CNN
-	1    4350 1650
+P 3650 1650
+F 0 "#PWR010" H 3650 1400 50  0001 C CNN
+F 1 "GND" H 3655 1477 50  0000 C CNN
+F 2 "" H 3650 1650 50  0001 C CNN
+F 3 "" H 3650 1650 50  0001 C CNN
+	1    3650 1650
 	1    0    0    -1
 $EndComp
@@
 L power:GND #PWR013
 U 1 1 5E57FDD5
-P 4800 1650
-F 0 "#PWR013" H 4800 1400 50  0001 C CNN
-F 1 "GND" H 4805 1477 50  0000 C CNN
-F 2 "" H 4800 1650 50  0001 C CNN
-F 3 "" H 4800 1650 50  0001 C CNN
-	1    4800 1650
-	1    0    0    -1
-$EndComp
-Wire Wire Line
-	3800 1650 3800 1550
-Wire Wire Line
-	4350 1550 4350 1650
-Wire Wire Line
-	4800 1650 4800 1550
+P 4100 1650
+F 0 "#PWR013" H 4100 1400 50  0001 C CNN
+F 1 "GND" H 4105 1477 50  0000 C CNN
+F 2 "" H 4100 1650 50  0001 C CNN
+F 3 "" H 4100 1650 50  0001 C CNN
+	1    4100 1650
+	1    0    0    -1
+$EndComp
+Wire Wire Line
+	3100 1650 3100 1550
+Wire Wire Line
+	3650 1550 3650 1650
+Wire Wire Line
+	4100 1650 4100 1550
 $Comp
 L Device:CP C6
@@
 F 0 "C6" H 5018 2346 50  0000 L CNN
 F 1 "10uF" H 5018 2255 50  0000 L CNN
-F 2 "Capacitor_Tantalum_SMD:CP_EIA-7260-38_AVX-R_Pad2.68x6.30mm_HandSolder" H 4938 2150 50  0001 C CNN
+F 2 "Capacitor_Tantalum_SMD:CP_EIA-3528-12_Kemet-T_Pad1.50x2.35mm_HandSolder" H 4938 2150 50  0001 C CNN
 F 3 "~" H 4900 2300 50  0001 C CNN
 	1    4900 2300
@@
 	7900 4050 8000 4050
 $Comp
-L Device:R R17
-U 1 1 5E5C944D
-P 4300 2800
-F 0 "R17" V 4093 2800 50  0000 C CNN
-F 1 "NP" V 4184 2800 50  0000 C CNN
-F 2 "Resistor_SMD:R_1206_3216Metric_Pad1.42x1.75mm_HandSolder" V 4230 2800 50  0001 C CNN
-F 3 "~" H 4300 2800 50  0001 C CNN
-	1    4300 2800
-	-1   0    0    1
-$EndComp
-Wire Wire Line
-	4300 2950 5150 2950
-Wire Wire Line
-	5150 2950 5150 2900
-Wire Wire Line
-	4300 2650 5150 2650
-Wire Wire Line
-	5150 2650 5150 2800
-$Comp
 L power:GND #PWR015
 U 1 1 5E5D022E
@@
 Connection ~ 4900 2100
 Wire Wire Line
-	3800 1050 4500 1050
-Wire Wire Line
-	4350 1250 4800 1250
-Connection ~ 4800 1250
+	3100 1050 3800 1050
+Wire Wire Line
+	3650 1250 4100 1250
+Connection ~ 4100 1250
 Connection ~ 6650 2300
 Wire Wire Line
@@
 Text Notes 3750 6650 1    50   ~ 0
 GND
+NoConn ~ 5150 2800
+NoConn ~ 5150 2900
+Wire Wire Line
+	4600 1700 5450 1700
 $EndSCHEMATC
